Commit message: Add full configuration for tool joint and tool link

File: ros2-code/src/rrbot_simulation_files/rrbot_description/gazebo/rrbot.gazebo.xacro (robot description, xacro)
@@ -28,4 +28,8 @@
       <material>Gazebo/Orange</material>
     </gazebo>
+    <!-- Tool Link (Link4) -->
+    <gazebo reference="${prefix}tool_link">
+      <material>Gazebo/Blue</material>
+    </gazebo>
   </xacro:macro>
 </robot>

File: ros2-code/src/rrbot_simulation_files/rrbot_description/ros2_control/rrbot.ros2_control.xacro (robot description, xacro)
@@ -11,5 +11,5 @@
       <hardware>
           <plugin>gazebo_ros2_control/GazeboSystem</plugin>
-        </hardware>
+      </hardware>
       <joint name="${prefix}joint1">
         <command_interface name="position">
@@ -46,4 +46,21 @@
         <state_interface name="effort"/>
       </joint>
+      <joint name="${prefix}tool_joint">
+        <command_interface name="position">
+          <param name="min">-10</param>
+          <param name="max">10</param>
+        </command_interface>
+        <command_interface name="velocity">
+          <param name="min">-10</param>
+          <param name="max">10</param>
+        </command_interface>
+        <command_interface name="effort">
+          <param name="min">-100</param>
+          <param name="max">100</param>
+        </command_interface>
+        <state_interface name="position"/>
+        <state_interface name="velocity"/>
+        <state_interface name="effort"/>
+      </joint>
     </ros2_control>
   </xacro:macro>

File: ros2-code/src/rrbot_simulation_files/rrbot_description/urdf/rrbot.urdf.xacro (robot description, xacro)
@@ -5,5 +5,5 @@
 https://github.com/ros-simulation/gazebo_ros_demos/blob/kinetic-devel/rrbot_description/urdf/rrbot.xacro
 -->
-<robot xmlns:xacro="http://www.ros.org/wiki/xacro" name="2dof_robot">
+<robot xmlns:xacro="http://www.ros.org/wiki/xacro" name="3dof_robot">
   <xacro:arg name="prefix" default="" />
   <!-- Import RRBot macro -->
@@ -24,4 +24,4 @@
   <xacro:rrbot_gazebo prefix="$(arg prefix)" />
   <xacro:rrbot_ros2_control
-    name="RRBot" prefix="$(arg prefix)" />
+    name="SCARA" prefix="$(arg prefix)" />
 </robot>

File: ros2-code/src/rrbot_simulation_files/rrbot_description/urdf/rrbot_description.urdf.xacro (robot description, xacro)
@@ -108,10 +108,9 @@
       </link>
       <joint name="${prefix}tool_joint" type="prismatic">
-        <origin xyz="0 0 1" rpy="0 1.5708 0" />
         <parent link="${prefix}link2"/>
         <child link="${prefix}tool_link" />
         <!-- Set limits of prismatic joint to -0.3 m to 0.3 m, 1000 N effort limit, velocity of 1 m/s  -->
         <limit lower="-1.5708" upper="1.5708" effort="1000" velocity="1"/>
-        <origin xyz="0 0 0" rpy="0 0 0"/>
+        <origin xyz="-2 0 1" rpy="0 1.5708 0" />
         <axis xyz="0 0 1"/>
         <dynamics damping="0.7"/>
@@ -130,7 +129,5 @@
             <box size="${prismatic_width} ${prismatic_width} ${height4}"/>
           </geometry>
-          <material name="blue">
-            <color rgba="0.0 0.0 1.0 0.5"/>
-          </material>
+          <material name="blue"/>
         </visual>
         <inertial>

Commit message: Change colors to green-grey-green-grey

File: ros2-code/src/rrbot_simulation_files/rrbot_description/gazebo/rrbot.gazebo.xacro (robot description, xacro)
@@ -14,5 +14,5 @@
     <!-- Link1 -->
     <gazebo reference="${prefix}base_link">
-      <material>Gazebo/Orange</material>
+      <material>Gazebo/Green</material>
     </gazebo>
     <!-- Link2 -->
@@ -20,5 +20,5 @@
       <mu1>0.2</mu1>
       <mu2>0.2</mu2>
-      <material>Gazebo/Black</material>
+      <material>Gazebo/Grey</material>
     </gazebo>
     <!-- Link3 -->
@@ -26,9 +26,9 @@
       <mu1>0.2</mu1>
       <mu2>0.2</mu2>
-      <material>Gazebo/Orange</material>
+      <material>Gazebo/Green</material>
     </gazebo>
     <!-- Tool Link (Link4) -->
     <gazebo reference="${prefix}tool_link">
-      <material>Gazebo/Blue</material>
+      <material>Gazebo/Grey</material>
     </gazebo>
   </xacro:macro>

File: ros2-code/src/rrbot_simulation_files/rrbot_description/urdf/rrbot_description.urdf.xacro (robot description, xacro)
@@ -32,5 +32,4 @@
         <box size="${width} ${width} ${height1}"/>
       </geometry>
-      <material name="orange"/>
     </visual>
     <inertial>
@@ -65,5 +64,4 @@
           <box size="${width} ${width} ${height2}"/>
         </geometry>
-        <material name="yellow"/>
       </visual>
       <inertial>
@@ -98,5 +96,4 @@
             <box size="${width} ${width} ${height3}"/>
           </geometry>
-          <material name="orange"/>
         </visual>
         <inertial>
@@ -131,5 +128,4 @@
             <box size="${prismatic_width} ${prismatic_width} ${height4}"/>
           </geometry>
-          <material name="blue"/>
         </visual>
         <inertial>

Commit message: Change greys to black

File: ros2-code/src/rrbot_simulation_files/rrbot_description/gazebo/rrbot.gazebo.xacro (robot description, xacro)
@@ -20,5 +20,5 @@
       <mu1>0.2</mu1>
       <mu2>0.2</mu2>
-      <material>Gazebo/Grey</material>
+      <material>Gazebo/Black</material>
     </gazebo>
     <!-- Link3 -->
@@ -30,5 +30,5 @@
     <!-- Tool Link (Link4) -->
     <gazebo reference="${prefix}tool_link">
-      <material>Gazebo/Grey</material>
+      <material>Gazebo/Black</material>
     </gazebo>
   </xacro:macro>
