Commit message: Change rotation axis of base link to z-axis, rotate it by 0.75 radians

File: ros2-code/src/rrbot_simulation_files/rrbot_description/urdf/rrbot_description.urdf.xacro (robot description, xacro)
@@ -42,6 +42,6 @@
       <parent link="${prefix}base_link"/>
       <child link="${prefix}link1"/>
-      <origin xyz="0 ${width} ${height1 - axel_offset}" rpy="0 1.5708 0"/>
-      <axis xyz="1 0 0"/>
+      <origin xyz="0 0 ${height1 + axel_offset}" rpy="0 1.5708 0.75"/>
+      <axis xyz="0 0 1"/>
       <dynamics damping="0.7"/>
     </joint>

Commit message: Set limits of revolute joint to -90deg to +90deg, 1000 N effort limit, velocity of 180 rad/s

File: ros2-code/src/rrbot_simulation_files/rrbot_description/urdf/rrbot_description.urdf.xacro (robot description, xacro)
@@ -39,7 +39,9 @@
       </inertial>
     </link>
-    <joint name="${prefix}joint1" type="continuous">
+    <joint name="${prefix}joint1" type="revolute">
       <parent link="${prefix}base_link"/>
       <child link="${prefix}link1"/>
+      <!-- Set limits of revolute joint to -90deg to +90deg, 1000 N effort limit, velocity of 180 rad/s  -->
+      <limit lower="-1.5708" upper="1.5708" effort="0.0" velocity="3.14159"/>
       <origin xyz="0 0 ${height1 + axel_offset}" rpy="0 1.5708 0.75"/>
       <axis xyz="0 0 1"/>

Commit message: Configure second joint

File: ros2-code/src/rrbot_simulation_files/rrbot_description/urdf/rrbot_description.urdf.xacro (robot description, xacro)
@@ -43,5 +43,5 @@
       <child link="${prefix}link1"/>
       <!-- Set limits of revolute joint to -90deg to +90deg, 1000 N effort limit, velocity of 180 rad/s  -->
-      <limit lower="-1.5708" upper="1.5708" effort="0.0" velocity="3.14159"/>
+      <limit lower="-1.5708" upper="1.5708" effort="1000" velocity="3.14159"/>
       <origin xyz="0 0 ${height1 + axel_offset}" rpy="0 1.5708 0.75"/>
       <axis xyz="0 0 1"/>
@@ -72,9 +72,11 @@
         </inertial>
       </link>
-      <joint name="${prefix}joint2" type="continuous">
+      <joint name="${prefix}joint2" type="revolute">
         <parent link="${prefix}link1"/>
         <child link="${prefix}link2"/>
-        <origin xyz="0 ${width} ${height2 - axel_offset*2}" rpy="0 0 0"/>
-        <axis xyz="1 0 0"/>
+        <!-- Set limits of revolute joint to -90deg to +90deg, 1000 N effort limit, velocity of 180 rad/s  -->
+        <limit lower="-1.5708" upper="1.5708" effort="1000" velocity="3.14159"/>
+        <origin xyz="0 0 ${height1 + axel_offset}" rpy="0 0 0"/>
+        <axis xyz="0 0 1"/>
         <dynamics damping="0.7"/>
       </joint>

Commit message: Get the second joint's placement right

File: ros2-code/src/rrbot_simulation_files/rrbot_description/urdf/rrbot_description.urdf.xacro (robot description, xacro)
@@ -77,5 +77,5 @@
         <!-- Set limits of revolute joint to -90deg to +90deg, 1000 N effort limit, velocity of 180 rad/s  -->
         <limit lower="-1.5708" upper="1.5708" effort="1000" velocity="3.14159"/>
-        <origin xyz="0 0 ${height1 + axel_offset}" rpy="0 0 0"/>
+        <origin xyz="${width * -1} 0 ${height2 - axel_offset*2}" rpy="0 0 0"/>
         <axis xyz="0 0 1"/>
         <dynamics damping="0.7"/>

Commit message: Rotate each joint offset by 45 deg, just to see how it looks

File: ros2-code/src/rrbot_simulation_files/rrbot_description/urdf/rrbot_description.urdf.xacro (robot description, xacro)
@@ -44,5 +44,5 @@
       <!-- Set limits of revolute joint to -90deg to +90deg, 1000 N effort limit, velocity of 180 rad/s  -->
       <limit lower="-1.5708" upper="1.5708" effort="1000" velocity="3.14159"/>
-      <origin xyz="0 0 ${height1 + axel_offset}" rpy="0 1.5708 0.75"/>
+      <origin xyz="0 0 ${height1 + axel_offset}" rpy="0 1.5708 0.785398"/>
       <axis xyz="0 0 1"/>
       <dynamics damping="0.7"/>
@@ -77,5 +77,5 @@
         <!-- Set limits of revolute joint to -90deg to +90deg, 1000 N effort limit, velocity of 180 rad/s  -->
         <limit lower="-1.5708" upper="1.5708" effort="1000" velocity="3.14159"/>
-        <origin xyz="${width * -1} 0 ${height2 - axel_offset*2}" rpy="0 0 0"/>
+        <origin xyz="${width * -1} 0 ${height2 - axel_offset*2}" rpy="0.785398 0 0"/>
         <axis xyz="0 0 1"/>
         <dynamics damping="0.7"/>

Commit message: Add TODO about revolution axis

File: ros2-code/src/rrbot_simulation_files/rrbot_description/urdf/rrbot_description.urdf.xacro (robot description, xacro)
@@ -78,5 +78,5 @@
         <limit lower="-1.5708" upper="1.5708" effort="1000" velocity="3.14159"/>
         <origin xyz="${width * -1} 0 ${height2 - axel_offset*2}" rpy="0.785398 0 0"/>
-        <axis xyz="0 0 1"/>
+        <axis xyz="0 0 1"/> <!-- TODO: We probably want to check this axis. If it follows the origin scheme above, we probably want to set this to -1 0 0 -->
         <dynamics damping="0.7"/>
       </joint>

Commit message: Set rotation axes of both revolute joints to -1 0 0

File: ros2-code/src/rrbot_simulation_files/rrbot_description/urdf/rrbot_description.urdf.xacro (robot description, xacro)
@@ -45,5 +45,5 @@
       <limit lower="-1.5708" upper="1.5708" effort="1000" velocity="3.14159"/>
       <origin xyz="0 0 ${height1 + axel_offset}" rpy="0 1.5708 0.785398"/>
-      <axis xyz="0 0 1"/>
+      <axis xyz="-1 0 0"/>
       <dynamics damping="0.7"/>
     </joint>
@@ -78,5 +78,5 @@
         <limit lower="-1.5708" upper="1.5708" effort="1000" velocity="3.14159"/>
         <origin xyz="${width * -1} 0 ${height2 - axel_offset*2}" rpy="0.785398 0 0"/>
-        <axis xyz="0 0 1"/> <!-- TODO: We probably want to check this axis. If it follows the origin scheme above, we probably want to set this to -1 0 0 -->
+        <axis xyz="-1 0 0"/>
         <dynamics damping="0.7"/>
       </joint>

Commit message: Set the home position of both joints to 0 in the z plane

File: ros2-code/src/rrbot_simulation_files/rrbot_description/urdf/rrbot_description.urdf.xacro (robot description, xacro)
@@ -44,5 +44,5 @@
       <!-- Set limits of revolute joint to -90deg to +90deg, 1000 N effort limit, velocity of 180 rad/s  -->
       <limit lower="-1.5708" upper="1.5708" effort="1000" velocity="3.14159"/>
-      <origin xyz="0 0 ${height1 + axel_offset}" rpy="0 1.5708 0.785398"/>
+      <origin xyz="0 0 ${height1 + axel_offset}" rpy="0 1.5708 0"/>
       <axis xyz="-1 0 0"/>
       <dynamics damping="0.7"/>
@@ -77,5 +77,5 @@
         <!-- Set limits of revolute joint to -90deg to +90deg, 1000 N effort limit, velocity of 180 rad/s  -->
         <limit lower="-1.5708" upper="1.5708" effort="1000" velocity="3.14159"/>
-        <origin xyz="${width * -1} 0 ${height2 - axel_offset*2}" rpy="0.785398 0 0"/>
+        <origin xyz="${width * -1} 0 ${height2 - axel_offset*2}" rpy="0 0 0"/>
         <axis xyz="-1 0 0"/>
         <dynamics damping="0.7"/>

Commit message: Double the width property for the whole robot

File: ros2-code/src/rrbot_simulation_files/rrbot_description/urdf/rrbot_description.urdf.xacro (robot description, xacro)
@@ -4,5 +4,5 @@
   <!-- Constants for robot dimensions -->
   <xacro:property name="mass" value="1" /> <!-- arbitrary value for mass -->
-  <xacro:property name="width" value="0.1" /> <!-- Square dimensions (widthxwidth) of beams -->
+  <xacro:property name="width" value="0.2" /> <!-- Square dimensions (widthxwidth) of beams -->
   <xacro:property name="height1" value="2" /> <!-- Link 1 -->
   <xacro:property name="height2" value="1" /> <!-- Link 2 -->

Commit message: Create a prismatic joint

File: ros2-code/src/rrbot_simulation_files/rrbot_description/urdf/rrbot_description.urdf.xacro (robot description, xacro)
@@ -8,4 +8,6 @@
   <xacro:property name="height2" value="1" /> <!-- Link 2 -->
   <xacro:property name="height3" value="1" /> <!-- Link 3 -->
+  <xacro:property name="height4" value="1" /> <!-- Link4 -->
+  <xacro:property name="prismatic_width" value="0.075" /> <!-- Thin width for prismatic link -->
   <xacro:property name="camera_link" value="0.05" /> <!-- Size of square 'camera' box -->
   <xacro:property name="axel_offset" value="0.05" /> <!-- Space btw top of beam and the each joint -->
@@ -104,13 +106,41 @@
             izz="${mass / 12.0 * (width*width + width*width)}"/>
           </inertial>
-        </link>
-        <joint name="${prefix}tool_joint" type="fixed">
-          <origin xyz="0 0 1" rpy="0 0 0" />
-          <parent link="${prefix}link2"/>
-          <child link="${prefix}tool_link" />
-        </joint>
-        <!-- Tool Link -->
-        <link name="${prefix}tool_link">
-        </link>
+      </link>
+      <joint name="${prefix}tool_joint" type="prismatic">
+        <origin xyz="0 0 1" rpy="0 1.5708 0" />
+        <parent link="${prefix}link2"/>
+        <child link="${prefix}tool_link" />
+        <!-- Set limits of prismatic joint to -0.3 m to 0.3 m, 1000 N effort limit, velocity of 1 m/s  -->
+        <limit lower="-1.5708" upper="1.5708" effort="1000" velocity="1"/>
+        <origin xyz="0 0 0" rpy="0 0 0"/>
+        <axis xyz="0 0 1"/>
+        <dynamics damping="0.7"/>
+      </joint>
+      <!-- Tool Link -->
+      <link name="${prefix}tool_link">
+        <collision>
+          <origin xyz="0 0 ${height4/2 - axel_offset}" rpy="0 0 0"/>
+          <geometry>
+            <box size="${prismatic_width} ${prismatic_width} ${height4}"/>
+          </geometry>
+        </collision>
+        <visual>
+          <origin xyz="0 0 ${height4/2 - axel_offset}" rpy="0 0 0"/>
+          <geometry>
+            <box size="${prismatic_width} ${prismatic_width} ${height4}"/>
+          </geometry>
+          <material name="blue">
+            <color rgba="0.0 0.0 1.0 0.5"/>
+          </material>
+        </visual>
+        <inertial>
+          <origin xyz="0 0 ${height4/2 - axel_offset}" rpy="0 0 0"/>
+          <mass value="${mass}"/>
+          <inertia
+            ixx="${mass / 12.0 * (prismatic_width*prismatic_width + height4*height4)}" ixy="0.0" ixz="0.0"
+            iyy="${mass / 12.0 * (height4*height4 + prismatic_width*prismatic_width)}" iyz="0.0"
+            izz="${mass / 12.0 * (prismatic_width*prismatic_width + prismatic_width*prismatic_width)}"/>
+          </inertial>
+      </link>
   </xacro:macro>
 </robot>

Commit message: Slightly improve origin and limits for tool joint

File: ros2-code/src/rrbot_simulation_files/rrbot_description/urdf/rrbot_description.urdf.xacro (robot description, xacro)
@@ -110,7 +110,7 @@
         <parent link="${prefix}link2"/>
         <child link="${prefix}tool_link" />
-        <!-- Set limits of prismatic joint to -0.3 m to 0.3 m, 1000 N effort limit, velocity of 1 m/s  -->
-        <limit lower="-1.5708" upper="1.5708" effort="1000" velocity="1"/>
-        <origin xyz="-2 0 1" rpy="0 1.5708 0" />
+        <!-- Set limits of prismatic joint -->
+        <limit lower="-0.19" upper="0.81" effort="1000" velocity="1"/>
+        <origin xyz="-0.81 0 0.9" rpy="0 1.5708 0" />
         <axis xyz="0 0 1"/>
         <dynamics damping="0.7"/>

Commit message: Raise the first joint a bit in order to prevent graphical glitch

File: ros2-code/src/rrbot_simulation_files/rrbot_description/urdf/rrbot_description.urdf.xacro (robot description, xacro)
@@ -46,5 +46,5 @@
       <!-- Set limits of revolute joint to -90deg to +90deg, 1000 N effort limit, velocity of 180 rad/s  -->
       <limit lower="-1.5708" upper="1.5708" effort="1000" velocity="3.14159"/>
-      <origin xyz="0 0 ${height1 + axel_offset}" rpy="0 1.5708 0"/>
+      <origin xyz="0 0 ${height1 + axel_offset*2}" rpy="0 1.5708 0"/>
       <axis xyz="-1 0 0"/>
       <dynamics damping="0.7"/>

Commit message: Improve origin of tool link

File: ros2-code/src/rrbot_simulation_files/rrbot_description/urdf/rrbot_description.urdf.xacro (robot description, xacro)
@@ -7,5 +7,5 @@
   <xacro:property name="height1" value="2" /> <!-- Link 1 -->
   <xacro:property name="height2" value="1" /> <!-- Link 2 -->
-  <xacro:property name="height3" value="1" /> <!-- Link 3 -->
+  <xacro:property name="height3" value="1.1" /> <!-- Link 3 -->
   <xacro:property name="height4" value="1" /> <!-- Link4 -->
   <xacro:property name="prismatic_width" value="0.075" /> <!-- Thin width for prismatic link -->
@@ -111,6 +111,6 @@
         <child link="${prefix}tool_link" />
         <!-- Set limits of prismatic joint -->
-        <limit lower="-0.19" upper="0.81" effort="1000" velocity="1"/>
-        <origin xyz="-0.81 0 0.9" rpy="0 1.5708 0" />
+        <limit lower="-10" upper="10" effort="1000" velocity="1"/>
+        <origin xyz="${axel_offset*2 + prismatic_width/2 + width - height4} 0 ${height3 - axel_offset*2}" rpy="0 1.5708 0" />
         <axis xyz="0 0 1"/>
         <dynamics damping="0.7"/>

Commit message: Define the prismatic offset property for reuse

File: ros2-code/src/rrbot_simulation_files/rrbot_description/urdf/rrbot_description.urdf.xacro (robot description, xacro)
@@ -8,8 +8,9 @@
   <xacro:property name="height2" value="1" /> <!-- Link 2 -->
   <xacro:property name="height3" value="1.1" /> <!-- Link 3 -->
-  <xacro:property name="height4" value="1" /> <!-- Link4 -->
   <xacro:property name="prismatic_width" value="0.075" /> <!-- Thin width for prismatic link -->
   <xacro:property name="camera_link" value="0.05" /> <!-- Size of square 'camera' box -->
   <xacro:property name="axel_offset" value="0.05" /> <!-- Space btw top of beam and the each joint -->
+  <xacro:property name="prismatic_offset" value="${axel_offset*2 + prismatic_width/2 + width}" /> <!-- This is the descended length in the zero position of the prismatic -->
+  <xacro:property name="height4" value="${1 + prismatic_offset}" /> <!-- Link4 -->
   <joint name="${prefix}base_joint" type="fixed">
     <xacro:insert_block name="origin" />
@@ -111,6 +112,6 @@
         <child link="${prefix}tool_link" />
         <!-- Set limits of prismatic joint -->
-        <limit lower="-10" upper="10" effort="1000" velocity="1"/>
-        <origin xyz="${axel_offset*2 + prismatic_width/2 + width - height4} 0 ${height3 - axel_offset*2}" rpy="0 1.5708 0" />
+        <limit lower="${prismatic_offset * -1}" upper="1.1" effort="1000" velocity="1"/>
+        <origin xyz="${prismatic_offset - height4} 0 ${height3 - axel_offset*2}" rpy="0 1.5708 0" />
         <axis xyz="0 0 1"/>
         <dynamics damping="0.7"/>

Commit message: Make the prismatic width thinner

File: ros2-code/src/rrbot_simulation_files/rrbot_description/urdf/rrbot_description.urdf.xacro (robot description, xacro)
@@ -8,5 +8,5 @@
   <xacro:property name="height2" value="1" /> <!-- Link 2 -->
   <xacro:property name="height3" value="1.1" /> <!-- Link 3 -->
-  <xacro:property name="prismatic_width" value="0.075" /> <!-- Thin width for prismatic link -->
+  <xacro:property name="prismatic_width" value="0.035" /> <!-- Thin width for prismatic link -->
   <xacro:property name="camera_link" value="0.05" /> <!-- Size of square 'camera' box -->
   <xacro:property name="axel_offset" value="0.05" /> <!-- Space btw top of beam and the each joint -->

Commit message: Define the width offset constant

File: ros2-code/src/rrbot_simulation_files/rrbot_description/urdf/rrbot_description.urdf.xacro (robot description, xacro)
@@ -11,5 +11,6 @@
   <xacro:property name="camera_link" value="0.05" /> <!-- Size of square 'camera' box -->
   <xacro:property name="axel_offset" value="0.05" /> <!-- Space btw top of beam and the each joint -->
-  <xacro:property name="prismatic_offset" value="${axel_offset*2 + prismatic_width/2 + width}" /> <!-- This is the descended length in the zero position of the prismatic -->
+  <xacro:property name="width_offset" value="0.037" /> <!-- Offset of prismatic link passing through the width -->
+  <xacro:property name="prismatic_offset" value="${axel_offset*2 + width_offset + width}" /> <!-- This is the descended length in the zero position of the prismatic -->
   <xacro:property name="height4" value="${1 + prismatic_offset}" /> <!-- Link4 -->
   <joint name="${prefix}base_joint" type="fixed">

Commit message: Set joint limits of joint1 and 2 to +/-150

File: ros2-code/src/rrbot_simulation_files/rrbot_description/urdf/rrbot_description.urdf.xacro (robot description, xacro)
@@ -45,6 +45,6 @@
       <parent link="${prefix}base_link"/>
       <child link="${prefix}link1"/>
-      <!-- Set limits of revolute joint to -90deg to +90deg, 1000 N effort limit, velocity of 180 rad/s  -->
-      <limit lower="-1.5708" upper="1.5708" effort="1000" velocity="3.14159"/>
+      <!-- Set limits of revolute joint to -150deg to +150deg, 1000 N effort limit, velocity of 180 rad/s  -->
+      <limit lower="-2.61799" upper="2.61799" effort="1000" velocity="3.14159"/>
       <origin xyz="0 0 ${height1 + axel_offset*2}" rpy="0 1.5708 0"/>
       <axis xyz="-1 0 0"/>
@@ -77,6 +77,6 @@
         <parent link="${prefix}link1"/>
         <child link="${prefix}link2"/>
-        <!-- Set limits of revolute joint to -90deg to +90deg, 1000 N effort limit, velocity of 180 rad/s  -->
-        <limit lower="-1.5708" upper="1.5708" effort="1000" velocity="3.14159"/>
+        <!-- Set limits of revolute joint to -150deg to +150deg, 1000 N effort limit, velocity of 180 rad/s  -->
+        <limit lower="-2.61799" upper="2.61799" effort="1000" velocity="3.14159"/>
         <origin xyz="${width * -1} 0 ${height2 - axel_offset*2}" rpy="0 0 0"/>
         <axis xyz="-1 0 0"/>

Commit message: Set joint limits as 0-90 and 0-150 for joints 1 and 2 respectively

File: ros2-code/src/rrbot_simulation_files/rrbot_description/urdf/rrbot_description.urdf.xacro (robot description, xacro)
@@ -45,6 +45,6 @@
       <parent link="${prefix}base_link"/>
       <child link="${prefix}link1"/>
-      <!-- Set limits of revolute joint to -150deg to +150deg, 1000 N effort limit, velocity of 180 rad/s  -->
-      <limit lower="-2.61799" upper="2.61799" effort="1000" velocity="3.14159"/>
+      <!-- Set limits of revolute joint to 0deg to +150deg, 1000 N effort limit, velocity of 180 rad/s  -->
+      <limit lower="0" upper="1.5708" effort="1000" velocity="3.14159"/>
       <origin xyz="0 0 ${height1 + axel_offset*2}" rpy="0 1.5708 0"/>
       <axis xyz="-1 0 0"/>
@@ -77,6 +77,6 @@
         <parent link="${prefix}link1"/>
         <child link="${prefix}link2"/>
-        <!-- Set limits of revolute joint to -150deg to +150deg, 1000 N effort limit, velocity of 180 rad/s  -->
-        <limit lower="-2.61799" upper="2.61799" effort="1000" velocity="3.14159"/>
+        <!-- Set limits of revolute joint to 0deg to +150deg, 1000 N effort limit, velocity of 180 rad/s  -->
+        <limit lower="0" upper="2.61799" effort="1000" velocity="3.14159"/>
         <origin xyz="${width * -1} 0 ${height2 - axel_offset*2}" rpy="0 0 0"/>
         <axis xyz="-1 0 0"/>

Commit message: Widen the limits of joint angles

File: ros2-code/src/rrbot_simulation_files/rrbot_description/urdf/rrbot_description.urdf.xacro (robot description, xacro)
@@ -45,6 +45,6 @@
       <parent link="${prefix}base_link"/>
       <child link="${prefix}link1"/>
-      <!-- Set limits of revolute joint to 0deg to +90deg, 1000 N effort limit, velocity of 180 rad/s  -->
-      <limit lower="0" upper="1.5708" effort="1000" velocity="3.14159"/>
+      <!-- Set limits of revolute joint to 0deg to +180deg, 1000 N effort limit, velocity of 180 rad/s  -->
+      <limit lower="0" upper="3.14159" effort="1000" velocity="3.14159"/>
       <origin xyz="0 0 ${height1 + axel_offset*2}" rpy="0 1.5708 0"/>
       <axis xyz="-1 0 0"/>
@@ -77,6 +77,6 @@
         <parent link="${prefix}link1"/>
         <child link="${prefix}link2"/>
-        <!-- Set limits of revolute joint to 0deg to +150deg, 1000 N effort limit, velocity of 180 rad/s  -->
-        <limit lower="0" upper="2.61799" effort="1000" velocity="3.14159"/>
+        <!-- Set limits of revolute joint to -150deg to +150deg, 1000 N effort limit, velocity of 180 rad/s  -->
+        <limit lower="-2.61799" upper="2.61799" effort="1000" velocity="3.14159"/>
         <origin xyz="${width * -1} 0 ${height2 - axel_offset*2}" rpy="0 0 0"/>
         <axis xyz="-1 0 0"/>

Commit message: Continue tuning, remove velocity limit

File: ros2-code/src/rrbot_simulation_files/rrbot_description/urdf/rrbot_description.urdf.xacro (robot description, xacro)
@@ -46,5 +46,5 @@
       <child link="${prefix}link1"/>
       <!-- Set limits of revolute joint to 0deg to +180deg, 1000 N effort limit, velocity of 180 rad/s  -->
-      <limit lower="0" upper="3.14159" effort="1000" velocity="3.14159"/>
+      <limit lower="0" upper="3.14159" effort="1000" velocity="6"/>
       <origin xyz="0 0 ${height1 + axel_offset*2}" rpy="0 1.5708 0"/>
       <axis xyz="-1 0 0"/>
@@ -78,5 +78,5 @@
         <child link="${prefix}link2"/>
         <!-- Set limits of revolute joint to -150deg to +150deg, 1000 N effort limit, velocity of 180 rad/s  -->
-        <limit lower="-2.61799" upper="2.61799" effort="1000" velocity="3.14159"/>
+        <limit lower="-2.61799" upper="2.61799" effort="1000" velocity="6"/>
         <origin xyz="${width * -1} 0 ${height2 - axel_offset*2}" rpy="0 0 0"/>
         <axis xyz="-1 0 0"/>
